File: Kicad/iMX6_BareBones.kicad_sch (KiCad schematic)
At the start: 0 parts

Commit message: For JLC DFM, added ground pours to L1 and L6. Updated soldermask expansion on U2 footprint.
Other:
- note added: "Revision 2 | 04/22/2026"
- note removed: "Revision 2 | 04/04/2026"
